Commit message: updated to enable gazebo launch

File: urdf/robot.urdf.xacro (robot description, xacro)
@@ -28,4 +28,7 @@
         </xacro:box_inertial>
     </link>
+    <gazebo reference= "chassis_link">
+        <material>Gazebo/Turquoise</material>
+    </gazebo>
     <!--Front left wheel Link-->
     <joint name="fl_wheel_joint" type="continuous">
@@ -51,4 +54,7 @@
         </xacro:cylinder_inertial>
     </link>
+    <gazebo reference= "fl_wheel_link">
+        <material>Gazebo/Black</material>
+    </gazebo>
     <!--Front right wheel Link-->
     <joint name="fr_wheel_joint" type="continuous">
@@ -74,4 +80,7 @@
         </xacro:cylinder_inertial>
     </link>
+    <gazebo reference= "fr_wheel_link">
+        <material>Gazebo/Black</material>
+    </gazebo>
     <!--Back left wheel Link-->
     <joint name="bl_wheel_joint" type="continuous">
@@ -97,4 +106,7 @@
         </xacro:cylinder_inertial>
     </link>
+    <gazebo reference= "bl_wheel_link">
+        <material>Gazebo/Black</material>
+    </gazebo>
     <!--Back right wheel Link-->
     <joint name="br_wheel_joint" type="continuous">
@@ -120,4 +132,6 @@
         </xacro:cylinder_inertial>
     </link>
-    <!--gazebo -->
+    <gazebo reference= "br_wheel_link">
+        <material>Gazebo/Black</material>
+    </gazebo>
 </robot>
